File: PowerBoard/PowerBoardDesign/RaspberryPi.sch (KiCad schematic (older format))
At the start: 1 part

Commit message: Update 1.2
Parts:
- added J?: Conn_01x02, symbol Connector_Generic:Conn_01x02
- added S?: IGT;MPU-6050, symbol PowerBoardComponents:IGT;MPU-6050
Connections:
- net at A?.3 (GPIO2/SDA): now also S?.3 (SDA)
- net at A?.5 (GPIO3/SCL): now also S?.2 (SCL)
- net at A?.7 (GPIO4/GPCKL0): now also S?.7 (INT)
- new net +5V: J?.2 (Pin_2), S?.1 (VCC)
- new net GND: J?.1 (Pin_1), S?.6 (AD0), S?.8 (GND)
Changed lines of the file:
@@
 	1    0    0    -1
 $EndComp
+$Comp
+L power:+5V #PWR?
+U 1 1 5DF3CAD1
+P 1700 800
+F 0 "#PWR?" H 1700 650 50  0001 C CNN
+F 1 "+5V" H 1715 973 50  0000 C CNN
+F 2 "" H 1700 800 50  0001 C CNN
+F 3 "" H 1700 800 50  0001 C CNN
+	1    1700 800
+	1    0    0    -1
+$EndComp
+Wire Wire Line
+	1700 800  1700 1000
+Wire Wire Line
+	1700 1000 1450 1000
+$Comp
+L PowerBoardComponents:IGT;MPU-6050 S?
+U 1 1 5DF3AD2E
+P 1200 1350
+F 0 "S?" H 1258 1965 50  0000 C CNN
+F 1 "IGT;MPU-6050" H 1258 1874 50  0000 C CNN
+F 2 "" H 1150 1500 50  0001 C CNN
+F 3 "" H 1200 1550 50  0001 C CNN
+	1    1200 1350
+	1    0    0    -1
+$EndComp
+$Comp
+L power:GND #PWR?
+U 1 1 5DF3ADF7
+P 1700 1900
+F 0 "#PWR?" H 1700 1650 50  0001 C CNN
+F 1 "GND" H 1705 1727 50  0000 C CNN
+F 2 "" H 1700 1900 50  0001 C CNN
+F 3 "" H 1700 1900 50  0001 C CNN
+	1    1700 1900
+	1    0    0    -1
+$EndComp
+Wire Wire Line
+	1450 1700 1700 1700
+Wire Wire Line
+	1700 1700 1700 1900
+Wire Wire Line
+	1450 1100 4650 1100
+Wire Wire Line
+	4650 1100 4650 3050
+Wire Wire Line
+	4650 3050 4900 3050
+Wire Wire Line
+	1450 1200 4750 1200
+Wire Wire Line
+	4750 1200 4750 2950
+Wire Wire Line
+	4750 2950 4900 2950
+Wire Wire Line
+	1450 1500 1700 1500
+Wire Wire Line
+	1700 1500 1700 1700
+Connection ~ 1700 1700
+Wire Wire Line
+	1450 1600 4550 1600
+Wire Wire Line
+	4550 1600 4550 3150
+Wire Wire Line
+	4550 3150 4900 3150
+$Comp
+L Connector_Generic:Conn_01x02 J?
+U 1 1 5DF4348B
+P 5550 2300
+F 0 "J?" H 5550 2000 50  0000 C CNN
+F 1 "Conn_01x02" H 5550 2100 50  0000 C CNN
+F 2 "" H 5550 2300 50  0001 C CNN
+F 3 "~" H 5550 2300 50  0001 C CNN
+	1    5550 2300
+	-1   0    0    1
+$EndComp
+$Comp
+L power:+5V #PWR?
+U 1 1 5DF47CDB
+P 5950 2150
+F 0 "#PWR?" H 5950 2000 50  0001 C CNN
+F 1 "+5V" H 5965 2323 50  0000 C CNN
+F 2 "" H 5950 2150 50  0001 C CNN
+F 3 "" H 5950 2150 50  0001 C CNN
+	1    5950 2150
+	1    0    0    -1
+$EndComp
+$Comp
+L power:GND #PWR?
+U 1 1 5DF48185
+P 5950 2350
+F 0 "#PWR?" H 5950 2100 50  0001 C CNN
+F 1 "GND" H 5955 2177 50  0000 C CNN
+F 2 "" H 5950 2350 50  0001 C CNN
+F 3 "" H 5950 2350 50  0001 C CNN
+	1    5950 2350
+	1    0    0    -1
+$EndComp
+Wire Wire Line
+	5750 2200 5950 2200
+Wire Wire Line
+	5950 2200 5950 2150
+Wire Wire Line
+	5950 2300 5950 2350
+Wire Wire Line
+	5750 2300 5950 2300
 $EndSCHEMATC
