File: PowerBoard/PowerBoardDesign/VoltageRegulation.sch (KiCad schematic (older format))
At the start: 4 parts

Commit message: Update 1.2
Parts:
- C?: value 33u -> 33µ
- C?: value 0.47u -> 0.47µ
Changed lines of the file:
@@
 P 3650 1400
 F 0 "C?" H 3768 1446 50  0000 L CNN
-F 1 "33u" H 3768 1355 50  0000 L CNN
+F 1 "33µ" H 3768 1355 50  0000 L CNN
 F 2 "" H 3688 1250 50  0001 C CNN
 F 3 "~" H 3650 1400 50  0001 C CNN
@@
 P 2550 1400
 F 0 "C?" H 2665 1446 50  0000 L CNN
-F 1 "0.47u" H 2665 1355 50  0000 L CNN
+F 1 "0.47µ" H 2665 1355 50  0000 L CNN
 F 2 "" H 2588 1250 50  0001 C CNN
 F 3 "~" H 2550 1400 50  0001 C CNN
